Commit message: get steered_wheel_base_controller running for debugging

File: zebROS_ws/src/frcrobot_description/urdf/frcrobot.xacro (robot description, xacro)
@@ -13,5 +13,5 @@
 					<box size="${swerve_box_size} ${swerve_box_size} ${swerve_box_size}"/>
 				</geometry>
-				<origin xyz="${x} ${y} -${base_height/2 + swerve_box_size/2}" rpy="0 0 0"/>
+				<origin xyz="0 0 0" rpy="0 0 0"/>
 				<material name="red">
 					<color rgba="1 0 0 1"/>
@@ -33,5 +33,5 @@
 			<parent link="base_link"/>
 			<child link="${prefix}_angle"/>
-			<origin xyz="0 0 0" rpy="0 0 0"/>
+			<origin xyz="${x} ${y} -${base_height/2 + swerve_box_size/2}" rpy="0 0 0"/>
 		</joint>
 		<joint name="${prefix}_angle_to_speed" type="continuous">
